Commit message: 2025/03/29 fixed format error in fishbot urdf

File: ch6/src/fishbot_description/urdf/first_robot.urdf.xacro (robot description, xacro)
@@ -28,5 +28,5 @@
             </material>
         </link>
-        <joint name="{imu_name}_joint" type="fixed">
+        <joint name="${imu_name}_joint" type="fixed">
             <parent link="base_link"/>
             <child link="${imu_name}_link"/>

File: ch6/src/fishbot_description/urdf/fishbot/fishbot.urdf.xacro (robot description, xacro)
@@ -5,5 +5,5 @@
     <xacro:include filename="$(find fishbot_description)/urdf/fishbot/sensor/laser.urdf.xacro"/>
     <xacro:include filename="$(find fishbot_description)/urdf/fishbot/sensor/camera.urdf.xacro"/>
-    <xacro:base_xacro length="0.12" radius="0.1">
+    <xacro:base_xacro length="0.12" radius="0.1"/>
     <xacro:imu_xacro xyz="0 0 0.02"/>
     <xacro:laser_xacro xyz="0 0 0.10"/>

File: ch6/src/fishbot_description/urdf/fishbot/sensor/laser.urdf.xacro (robot description, xacro)
@@ -22,5 +22,5 @@
                 <origin xyz="0.0 0.0 0.0" rpy="0.0 0.0 0.0"/>
                 <geometry>
-                    <cylinder length="${length}" radius="${radius}"/>
+                    <cylinder length="0.02" radius="$0.02"/>
                 </geometry>
                 <material name="green">
