Commit message: 2025/03/30 add inertail property to all the component.

File: ch6/src/fishbot_description/urdf/fishbot/base.urdf.xacro (robot description, xacro)
@@ -1,10 +1,17 @@
 <?xml version="1.0"?>
 <robot xmlns:xacro="http://www.ros.org/wiki/xacro">
+    <xacro:include filename="$(find fishbot_description)/urdf/fishbot/common_inertia.xacro"/>
     <xacro:macro name="base_xacro" params="length radius">
+        <link name="base_footprint" />
+        <joint name="base_joint" type="fixed">
+            <parent link="base_footprint"/>
+            <child link="base_link"/>
+            <origin xyz="0.0 0.0 ${length/2.0 + 0.032 - 0.001}" rpy="0.0 0.0 0.0"/>
+        </joint>
         <link name="base_link">
             <visual>
                 <origin xyz="0.0 0.0 0.0" rpy="0.0 0.0 0.0"/>
                 <geometry>
-                    <cylinder length="${length}" radius="${radius}"/>
+                    <cylinder length="${length}" radius="${length}"/>
                 </geometry>
                 <material name="white">
@@ -12,4 +19,11 @@
                 </material>
             </visual>
+            <collision>
+                <origin xyz="0.0 0.0 0.0" rpy="0.0 0.0 0.0"/>
+                <geometry>
+                    <cylinder length="${length}" radius="${length}"/>
+                </geometry>
+            </collision>
+            <xacro:cylinder_inertia m="1.0" r="${radius}" h="${length}"/>
         </link>
     </xacro:macro>

File: ch6/src/fishbot_description/urdf/fishbot/fishbot.urdf.xacro (robot description, xacro)
@@ -5,7 +5,16 @@
     <xacro:include filename="$(find fishbot_description)/urdf/fishbot/sensor/laser.urdf.xacro"/>
     <xacro:include filename="$(find fishbot_description)/urdf/fishbot/sensor/camera.urdf.xacro"/>
+    <xacro:include filename="$(find fishbot_description)/urdf/fishbot/actuator/wheel.urdf.xacro"/>
+    <xacro:include filename="$(find fishbot_description)/urdf/fishbot/actuator/caster.urdf.xacro"/>
+    <!-- base params -->
     <xacro:base_xacro length="0.12" radius="0.1"/>
+    <!-- sensor params -->
     <xacro:imu_xacro xyz="0 0 0.02"/>
     <xacro:laser_xacro xyz="0 0 0.10"/>
     <xacro:camera_xacro xyz="0.10 0 0.075"/>
+    <!-- actuator params -->
+    <xacro:wheel_xacro wheel_name="left" xyz="0.0 0.10 -0.06"/>
+    <xacro:wheel_xacro wheel_name="right" xyz="0.0 -0.10 -0.06"/>
+    <xacro:caster_xacro caster_name="front" xyz="0.08 0.0 -0.076"/>
+    <xacro:caster_xacro caster_name="back" xyz="-0.08 0.0 -0.076"/>
 </robot>

File: ch6/src/fishbot_description/urdf/fishbot/sensor/camera.urdf.xacro (robot description, xacro)
@@ -13,4 +13,11 @@
                 </material>
             </visual>
+            <collision>
+                <origin xyz="0.0 0.0 0.0" rpy="0.0 0.0 0.0"/>
+                <geometry>
+                    <box size="0.02 0.10 0.02"/>
+                </geometry>
+            </collision>
+            <xacro:box_inertia m="1.0" w="0.02" h="0.10" d="0.02"/>
         </link>
         <joint name="camera_joint" type="fixed">

File: ch6/src/fishbot_description/urdf/fishbot/sensor/imu.urdf.xacro (robot description, xacro)
@@ -12,4 +12,11 @@
                 </material>
             </visual>
+            <collision>
+                <origin xyz="0.0 0.0 0.0" rpy="0.0 0.0 0.0"/>
+                <geometry>
+                    <box size="0.02 0.02 0.02"/>
+                </geometry>
+            </collision>
+            <xacro:box_inertia m="1.0" w="0.02" h="0.02" d="0.02"/>
         </link>
         <joint name="imu_joint" type="fixed">

File: ch6/src/fishbot_description/urdf/fishbot/sensor/laser.urdf.xacro (robot description, xacro)
@@ -12,4 +12,11 @@
                 </material>
             </visual>
+            <collision>
+                <origin xyz="0.0 0.0 0.0" rpy="0.0 0.0 0.0"/>
+                <geometry>
+                    <cylinder length="0.10" radius="0.01"/>
+                </geometry>
+            </collision>
+            <xacro:cylinder_inertia m="1.0" r="0.01" h="0.10"/>
         </link>
         <joint name="laser_cylinder_joint" type="fixed">
@@ -22,5 +29,5 @@
                 <origin xyz="0.0 0.0 0.0" rpy="0.0 0.0 0.0"/>
                 <geometry>
-                    <cylinder length="0.02" radius="$0.02"/>
+                    <cylinder length="0.02" radius="0.02"/>
                 </geometry>
                 <material name="green">
@@ -28,4 +35,11 @@
                 </material>
             </visual>
+            <collision>
+                <origin xyz="0.0 0.0 0.0" rpy="0.0 0.0 0.0"/>
+                <geometry>
+                    <cylinder length="0.02" radius="0.02"/>
+                </geometry>
+            </collision>
+            <xacro:cylinder_inertia m="1.0" r="0.02" h="0.02"/>
         </link>
         <joint name="laser_joint" type="fixed">
