Commit message: 2025/03/30 add gazerbo config.

File: ch6/src/fishbot_description/urdf/fishbot/actuator/caster.urdf.xacro (robot description, xacro)
@@ -29,4 +29,11 @@
             <axis xyz="0.0 0.0 0.0"/>
         </joint>
+        <gazebo reference="${caster_name}_caster_link">
+            <!-- 切向摩擦系数、 法向摩擦系数、接触刚度系数、阻尼系数 -->
+            <mu1 value="0.0"/>
+            <mu2 value="0.0"/>
+            <kp value="1000000000.0"/>
+            <kd value="1.0"/>
+        </gazebo>
     </xacro:macro>
 </robot>

File: ch6/src/fishbot_description/urdf/fishbot/actuator/wheel.urdf.xacro (robot description, xacro)
@@ -29,4 +29,11 @@
             <axis xyz="0.0 1.0 0.0"/>
         </joint>
+        <gazebo reference="${wheel_name}_wheel_link">
+            <!-- 切向摩擦系数、 法向摩擦系数、接触刚度系数、阻尼系数 -->
+            <mu1 value="20.0"/>
+            <mu2 value="20.0"/>
+            <kp value="1000000000.0"/>
+            <kd value="1.0"/>
+        </gazebo>
     </xacro:macro>
 </robot>

File: ch6/src/fishbot_description/urdf/fishbot/sensor/laser.urdf.xacro (robot description, xacro)
@@ -2,4 +2,14 @@
 <robot xmlns:xacro="http://www.ros.org/wiki/xacro">
     <xacro:macro name="laser_xacro" params="xyz">
+        <gazebo reference="laser_cylinder_link">
+            <material>
+                Gazebo/Black
+            </material>
+        </gazebo>
+        <gazebo reference="laser_link">
+            <material>
+                Gazebo/Black
+            </material>
+        </gazebo>
         <link name="laser_cylinder_link">
             <visual>
