Commit message: 2025/03/30 finished gazebo control, implement teleop control.

File: ch6/src/fishbot_description/urdf/fishbot/actuator/wheel.urdf.xacro (robot description, xacro)
@@ -30,4 +30,5 @@
         </joint>
         <gazebo reference="${wheel_name}_wheel_link">
+            <material>Gazebo/Black</material>
             <!-- 切向摩擦系数、 法向摩擦系数、接触刚度系数、阻尼系数 -->
             <mu1 value="20.0"/>

File: ch6/src/fishbot_description/urdf/fishbot/fishbot.urdf.xacro (robot description, xacro)
@@ -7,4 +7,5 @@
     <xacro:include filename="$(find fishbot_description)/urdf/fishbot/actuator/wheel.urdf.xacro"/>
     <xacro:include filename="$(find fishbot_description)/urdf/fishbot/actuator/caster.urdf.xacro"/>
+    <xacro:include filename="$(find fishbot_description)/urdf/fishbot/plugins/gazebo_control_plugin.xacro"/>
     <!-- base params -->
     <xacro:base_xacro length="0.12" radius="0.1"/>
@@ -18,3 +19,4 @@
     <xacro:caster_xacro caster_name="front" xyz="0.08 0.0 -0.076"/>
     <xacro:caster_xacro caster_name="back" xyz="-0.08 0.0 -0.076"/>
+    <xacro:gazebo_control_plugin/>
 </robot>

File: ch6/src/fishbot_description/urdf/fishbot/plugins/gazebo_control_plugin.xacro (robot description, xacro)
@@ -11,6 +11,6 @@
                 <update_rate>30</update_rate>
                 <!-- wheels -->
-                <left_join>left_wheel_joint</left_join>
-                <right_join>right_wheel_joint</right_join>
+                <left_joint>left_wheel_joint</left_joint>
+                <right_joint>right_wheel_joint</right_joint>
                 <!-- kinematic -->
                 <wheel_separation>0.2</wheel_separation>

File: ch6/src/fishbot_description/urdf/fishbot/sensor/camera.urdf.xacro (robot description, xacro)
@@ -2,4 +2,7 @@
 <robot xmlns:xacro="http://www.ros.org/wiki/xacro">
     <xacro:macro name="camera_xacro" params="xyz">
+    <gazebo reference="camera_link">
+        <material>Gazebo/Black</material>
+    </gazebo>
         <!-- camera module-->
         <link name="camera_link">
